Commit message: Add 3d robot

File: models/point_mass_robot_3d.urdf (robot description, URDF)
Before this commit: robot pointmass2d, 4 links, 3 joints
Links:
- added link dummy3
Joints:
- removed joint fixed_dummy2_robot
- added joint fixed_dummy3_robot: type fixed, parent dummy3, child robot, origin xyz=0 0 0, axis 0 0 0
- added joint p_joint_z: type prismatic, parent dummy2, child dummy3, origin xyz=0 0 0, axis 0 0 1, limit lower=-1.0 upper=1.0 effort=1.0 velocity=5.0
